File: elec/Kicad/LCD.kicad_sch (KiCad schematic)
At the start: 0 parts

Commit message: merci charles de m'aider a nous aider
Other:
- note added: "LCD SPI idéalement"
Changed lines of the file:
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@@
 	(generator_version "8.0")
 	(paper "A4")
+	(text "LCD SPI idéalement\n"
+		(exclude_from_sim no)
+		(at 48.006 22.606 0)
+		(effects
+			(font
+				(size 1.27 1.27)
+			)
+		)
+	)
 )

Commit message: j'ai fait l'écran
Parts:
- added C14, C16: 0.1uF, symbol Device:C
- added J5: Conn_01x13_Shielded, Connector_FFC-FPC:Hirose_FH12-13S-0.5SH_1x13-1MP_P0.50mm_Horizontal, symbol Connector_Generic_Shielded:Conn_01x13_Shielded
- added Q4: SS8050, Package_TO_SOT_SMD:SOT-23, symbol Transistor_BJT:SS8050
- added R21: 10, symbol Device:R
- added R26: 10K, symbol Device:R
- added R27: 1K, symbol Device:R
Connections:
- new net: Q4.1 (B), R26.1, R27.1
- new net: C16.1, J5.12 (Pin_12)
- new net: Q4.3 (C), R21.1
- new net +3.3V: C14.1, J5.10 (Pin_10), R26.2
- new net BL_LCD: R27.2
- new net CS_LCD: J5.7 (Pin_7)
- new net GND: C14.2, C16.2, J5.13 (Pin_13), J5.8 (Pin_8), Q4.2 (E)
- new net LEDK: J5.11 (Pin_11), R21.2
- new net RESET_LCD: J5.6 (Pin_6)
- new net RS_LCD: J5.5 (Pin_5)
- new net SPI1_MOSI: J5.3 (Pin_3)
- new net SPI1_SCK: J5.4 (Pin_4)
- no-connect marks 0 -> 4
Other:
- note added: "3.3V"
- note added: "CS"
- note added: "GND"
- note added: "LEDA"
- note added: "LEDK"
- note added: "Le LCD serait un 1.14" sur AliExpress LCD DRIVER = ST7789 Resolution: 240 x 135 pixels Dimension: 31 x 18 mm longeur du Film FCP = 15.85 mm largeur du Film FCP = 12.4 mm"
- note added: "NC"
- note added: "RESET"
- note added: "RS"
- note added: "RS = Register Select elle indique si on envoie une commande (0) ou une donnée (1) RESET = quand elle est a 0, on reset le lcd driver LEDK = anode de l'écran, elle fourni l'éclairage (doit être a 1) LEDA = cathode de l'écran, doit être au GND C'est ce que chat me dit pcq j'ai méga la fleme de vérifier live sinon la schématic est basé sur celle d'un breakout board so i guess we good"
- note added: "SCL (CLK)"
- note added: "SDA (MOSI)"

Commit message: va falloir faire le PCB soon
Parts:
- added C19, C20: 100nF, symbol Device:C
- added C21: 1uF, symbol Device:C
- added C22: 2.2uF, symbol Device:C
- added U11: MMC5633NJL, Package_BGA:WLP-4_0.86x0.86mm_P0.4mm, symbol Sensor_Magnetic:MMC5633NJL
- added U2: BMI160, Package_LGA:Bosch_LGA-14_3x2.5mm_P0.5mm, symbol Sensor_Motion:BMI160
- added U8: LTR-303ALS-01, OptoDevice:Lite-On_LTR-303ALS-01, symbol Sensor_Optical:LTR-303ALS-01
Connections:
- net +3.3V: now also C19.1, C20.1, U2.5 (VDDIO), U2.8 (VDD)
- net GND: now also C19.2, C20.2, C21.2, C22.2, U11.A1 (VSA), U2.1 (SDO), U2.6 (GNDIO), U2.7 (GND), U8.3 (GND)
- new net: C22.1, U11.B1 (VDD)
- new net: C21.1, U8.1 (VDD)
- new net I2C1_SCL: U11.B2 (SDA), U2.13 (SCx), U8.4 (SCL)
- new net I2C1_SDA: U11.A2 (SCL), U2.14 (SDx), U8.6 (SDA)
- no-connect marks 4 -> 12
Other:
- note added: "BMI160 (6-axis)"
- note added: "For default I2C addr (SD0 to GND)"
- note added: "I2C address=0x29"
- note added: "I2C address=0x30"
- note added: "I2C address=0x68"
- note added: "LUX Sensor"
- note added: "Magnetometre"

Commit message: add a few footprint
Parts:
- C14, C16: value 0.1uF -> 100nF; footprint (none) -> Capacitor_SMD:C_0603_1608Metric_Pad1.08x0.95mm_HandSolder
- C19, C20, C21, C22: footprint (none) -> Capacitor_SMD:C_0603_1608Metric_Pad1.08x0.95mm_HandSolder
- R21, R26, R27: footprint (none) -> Resistor_SMD:R_0603_1608Metric_Pad0.98x0.95mm_HandSolder
Other:
- moved on the sheet: Q4, R21, R26, R27
Changed lines of the file:
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@@
 	)
 	(junction
-		(at 78.74 96.52)
+		(at 52.07 100.33)
 		(diameter 0)
 		(color 0 0 0 0)
@@
 	(wire
 		(pts
-			(xy 71.12 96.52) (xy 78.74 96.52)
+			(xy 44.45 100.33) (xy 52.07 100.33)
 		)
 		(stroke
@@
 	(wire
 		(pts
-			(xy 91.44 101.6) (xy 97.79 101.6)
-		)
-		(stroke
-			(width 0)
-			(type default)
-		)
-	)
-	(wire
-		(pts
-			(xy 78.74 96.52) (xy 83.82 96.52)
-		)
-		(stroke
-			(width 0)
-			(type default)
-		)
-	)
-	(wire
-		(pts
-			(xy 97.79 101.6) (xy 97.79 106.68)
+			(xy 64.77 105.41) (xy 71.12 105.41)
+		)
+		(stroke
+			(width 0)
+			(type default)
+		)
+	)
+	(wire
+		(pts
+			(xy 52.07 100.33) (xy 57.15 100.33)
+		)
+		(stroke
+			(width 0)
+			(type default)
+		)
+	)
+	(wire
+		(pts
+			(xy 71.12 105.41) (xy 71.12 110.49)
 		)
 		(stroke
@@
 	(wire
 		(pts
-			(xy 91.44 86.36) (xy 97.79 86.36)
+			(xy 64.77 90.17) (xy 71.12 90.17)
 		)
 		(stroke
@@
 	(wire
 		(pts
-			(xy 78.74 82.55) (xy 78.74 83.82)
+			(xy 52.07 86.36) (xy 52.07 87.63)
 		)
 		(stroke
@@
 	(wire
 		(pts
-			(xy 78.74 91.44) (xy 78.74 96.52)
+			(xy 52.07 95.25) (xy 52.07 100.33)
 		)
 		(stroke
@@
 	(wire
 		(pts
-			(xy 91.44 91.44) (xy 91.44 86.36)
+			(xy 64.77 95.25) (xy 64.77 90.17)
 		)
 		(stroke
@@
 	(global_label "LEDK"
 		(shape input)
-		(at 105.41 86.36 0)
+		(at 78.74 90.17 0)
 		(fields_autoplaced yes)
 		(effects
@@
 		)
 		(property "Intersheetrefs" "${INTERSHEET_REFS}"
-			(at 111.5716 86.36 0)
+			(at 84.9016 90.17 0)
 			(effects
 				(font
@@
 	(global_label "BL_LCD"
 		(shape input)
-		(at 63.5 96.52 180)
+		(at 36.83 100.33 180)
 		(fields_autoplaced yes)
 		(effects
@@
 		)
 		(property "Intersheetrefs" "${INTERSHEET_REFS}"
-			(at 55.645 96.52 0)
+			(at 28.975 100.33 0)
 			(effects
 				(font
@@
 			)
 		)
-		(property "Footprint" ""
+		(property "Footprint" "Capacitor_SMD:C_0603_1608Metric_Pad1.08x0.95mm_HandSolder"
 			(at 239.7252 134.62 0)
 			(effects
@@
 			)
 		)
-		(property "Footprint" ""
+		(property "Footprint" "Capacitor_SMD:C_0603_1608Metric_Pad1.08x0.95mm_HandSolder"
 			(at 134.3152 139.7 0)
 			(effects
@@
 			)
 		)
-		(property "Datasheet" "~"
+		(property "Datasheet" "https://www.digikey.ca/en/products/detail/yageo/CC0603KRX7R7BB104/302822"
 			(at 133.35 135.89 0)
 			(effects
@@
 	(symbol
 		(lib_id "Device:R")
-		(at 78.74 87.63 180)
+		(at 52.07 91.44 180)
 		(unit 1)
 		(exclude_from_sim no)
@@
 		(fields_autoplaced yes)
 		(property "Reference" "R26"
-			(at 81.28 86.3599 0)
+			(at 54.61 90.1699 0)
 			(effects
 				(font
@@
 		)
 		(property "Value" "10K"
-			(at 81.28 88.8999 0)
+			(at 54.61 92.7099 0)
 			(effects
 				(font
@@
 			)
 		)
-		(property "Footprint" ""
-			(at 80.518 87.63 90)
+		(property "Footprint" "Resistor_SMD:R_0603_1608Metric_Pad0.98x0.95mm_HandSolder"
+			(at 53.848 91.44 90)
 			(effects
 				(font
@@
 		)
 		(property "Datasheet" "~"
-			(at 78.74 87.63 0)
+			(at 52.07 91.44 0)
 			(effects
 				(font
@@
 		)
 		(property "Description" "Resistor"
-			(at 78.74 87.63 0)
+			(at 52.07 91.44 0)
 			(effects
 				(font
@@
 			)
 		)
-		(property "Value" "0.1uF"
+		(property "Value" "100nF"
 			(at 34.29 69.8499 0)
 			(effects
@@
 			)
 		)
-		(property "Footprint" ""
+		(property "Footprint" "Capacitor_SMD:C_0603_1608Metric_Pad1.08x0.95mm_HandSolder"
 			(at 31.4452 72.39 0)
 			(effects
@@
 			)
 		)
-		(property "Value" "0.1uF"
+		(property "Value" "100nF"
 			(at 46.99 69.8499 0)
 			(effects
@@
 			)
 		)
-		(property "Footprint" ""
+		(property "Footprint" "Capacitor_SMD:C_0603_1608Metric_Pad1.08x0.95mm_HandSolder"
 			(at 44.1452 72.39 0)
 			(effects
@@
 	(symbol
 		(lib_id "power:GND")
-		(at 97.79 106.68 0)
+		(at 71.12 110.49 0)
 		(unit 1)
 		(exclude_from_sim no)
@@
 		(fields_autoplaced yes)
 		(property "Reference" "#PWR013"
-			(at 97.79 113.03 0)
+			(at 71.12 116.84 0)
 			(effects
 				(font
@@
 		)
 		(property "Value" "GND"
-			(at 97.79 111.76 0)
+			(at 71.12 115.57 0)
 			(effects
 				(font
@@
 		)
 		(property "Footprint" ""
-			(at 97.79 106.68 0)
+			(at 71.12 110.49 0)
 			(effects
 				(font
@@
 		)
 		(property "Datasheet" ""
-			(at 97.79 106.68 0)
+			(at 71.12 110.49 0)
 			(effects
 				(font
@@
 		)
 		(property "Description" "Power symbol creates a global label with name \"GND\" , ground"
-			(at 97.79 106.68 0)
+			(at 71.12 110.49 0)
 			(effects
 				(font
@@
 			)
 		)
-		(property "Footprint" ""
+		(property "Footprint" "Capacitor_SMD:C_0603_1608Metric_Pad1.08x0.95mm_HandSolder"
 			(at 195.2752 86.36 0)
 			(effects
@@
 	(symbol
 		(lib_id "Device:R")
-		(at 67.31 96.52 270)
+		(at 40.64 100.33 270)
 		(unit 1)
 		(exclude_from_sim no)
@@
 		(fields_autoplaced yes)
 		(property "Reference" "R27"
-			(at 67.31 90.17 90)
+			(at 40.64 93.98 90)
 			(effects
 				(font
@@
 		)
 		(property "Value" "1K"
-			(at 67.31 92.71 90)
-			(effects
-				(font
-					(size 1.27 1.27)
-				)
-			)
-		)
-		(property "Footprint" ""
-			(at 67.31 94.742 90)
+			(at 40.64 96.52 90)
+			(effects
+				(font
+					(size 1.27 1.27)
+				)
+			)
+		)
+		(property "Footprint" "Resistor_SMD:R_0603_1608Metric_Pad0.98x0.95mm_HandSolder"
+			(at 40.64 98.552 90)
 			(effects
 				(font
@@
 		)
 		(property "Datasheet" "~"
-			(at 67.31 96.52 0)
+			(at 40.64 100.33 0)
 			(effects
 				(font
@@
 		)
 		(property "Description" "Resistor"
-			(at 67.31 96.52 0)
+			(at 40.64 100.33 0)
 			(effects
 				(font
@@
 			)
 		)
-		(property "Footprint" ""
+		(property "Footprint" "Capacitor_SMD:C_0603_1608Metric_Pad1.08x0.95mm_HandSolder"
 			(at 120.3452 139.7 0)
 			(effects
@@
 			)
 		)
-		(property "Datasheet" "~"
+		(property "Datasheet" "https://www.digikey.ca/en/products/detail/yageo/CC0603KRX7R7BB104/302822"
 			(at 119.38 135.89 0)
 			(effects
@@
 	(symbol
 		(lib_id "Transistor_BJT:SS8050")
-		(at 88.9 96.52 0)
+		(at 62.23 100.33 0)
 		(unit 1)
 		(exclude_from_sim no)
@@
 		(fields_autoplaced yes)
 		(property "Reference" "Q4"
-			(at 93.98 95.2499 0)
+			(at 67.31 99.0599 0)
 			(effects
 				(font
@@
 		)
 		(property "Value" "SS8050"
-			(at 93.98 97.7899 0)
+			(at 67.31 101.5999 0)
 			(effects
 				(font
@@
 		)
 		(property "Footprint" "Package_TO_SOT_SMD:SOT-23"
-			(at 93.98 103.886 0)
+			(at 67.31 107.696 0)
 			(effects
 				(font
@@
 		)
 		(property "Datasheet" "http://www.secosgmbh.com/datasheet/products/SSMPTransistor/SOT-23/SS8050.pdf"
-			(at 93.98 101.346 0)
+			(at 67.31 105.156 0)
 			(effects
 				(font
@@
 		)
 		(property "Description" "General Purpose NPN Transistor, 1.5A Ic, 25V Vce, SOT-23"
-			(at 122.936 98.806 0)
+			(at 96.266 102.616 0)
 			(effects
 				(font
@@
 	(symbol
 		(lib_id "power:+3.3V")
-		(at 78.74 82.55 0)
+		(at 52.07 86.36 0)
 		(unit 1)
 		(exclude_from_sim no)
@@
 		(fields_autoplaced yes)
 		(property "Reference" "#PWR014"
-			(at 78.74 86.36 0)
+			(at 52.07 90.17 0)
 			(effects
 				(font
@@
 		)
 		(property "Value" "+3.3V"
-			(at 78.74 77.47 0)
+			(at 52.07 81.28 0)
 			(effects
 				(font
@@
 		)
 		(property "Footprint" ""
-			(at 78.74 82.55 0)
+			(at 52.07 86.36 0)
 			(effects
 				(font
@@
 		)
 		(property "Datasheet" ""
-			(at 78.74 82.55 0)
+			(at 52.07 86.36 0)
 			(effects
 				(font
@@
 		)
 		(property "Description" "Power symbol creates a global label with name \"+3.3V\""
-			(at 78.74 82.55 0)
+			(at 52.07 86.36 0)
 			(effects
 				(font
@@
 	(symbol
 		(lib_id "Device:R")
-		(at 101.6 86.36 90)
+		(at 74.93 90.17 90)
 		(unit 1)
 		(exclude_from_sim no)
@@
 		(fields_autoplaced yes)
 		(property "Reference" "R21"
-			(at 101.6 80.01 90)
+			(at 74.93 83.82 90)
 			(effects
 				(font
@@
 		)
 		(property "Value" "10"
-			(at 101.6 82.55 90)
-			(effects
-				(font
-					(size 1.27 1.27)
-				)
-			)
-		)
-		(property "Footprint" ""
-			(at 101.6 88.138 90)
+			(at 74.93 86.36 90)
+			(effects
+				(font
+					(size 1.27 1.27)
+				)
+			)
+		)
+		(property "Footprint" "Resistor_SMD:R_0603_1608Metric_Pad0.98x0.95mm_HandSolder"
+			(at 74.93 91.948 90)
 			(effects
 				(font
@@
 		)
 		(property "Datasheet" "~"
-			(at 101.6 86.36 0)
+			(at 74.93 90.17 0)
 			(effects
 				(font
@@
 		)
 		(property "Description" "Resistor"
-			(at 101.6 86.36 0)
-			(effects
-				(font
+			(at 74.93 90.17 0)
+			(effects
+				(font

Commit message: formation torture
Connections:
- net +3.3V: now also C21.1, C22.1, U11.B1 (VDD), U8.1 (VDD)
Changed lines of the file:
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@@
+	)
+	(junction
+		(at 167.64 72.39)
+		(diameter 0)
+		(color 0 0 0 0)
 	)
 	(junction
@@
 	)
 	(junction
+		(at 213.36 123.19)
+		(diameter 0)
+		(color 0 0 0 0)
+	)
+	(junction
 		(at 133.35 132.08)
 		(diameter 0)
@@
 	(text "I2C address=0x30\n"
 		(exclude_from_sim no)
-		(at 207.264 119.38 0)
+		(at 200.914 118.11 0)
 		(effects
 			(font
@@
 	(text "I2C address=0x29\n"
 		(exclude_from_sim no)
-		(at 169.164 70.612 0)
+		(at 151.13 68.58 0)
 		(effects
 			(font
@@
 	)
 	(symbol
+		(lib_id "power:+3.3V")
+		(at 167.64 72.39 0)
+		(unit 1)
+		(exclude_from_sim no)
+		(in_bom yes)
+		(on_board yes)
+		(dnp no)
+		(fields_autoplaced yes)
+		(property "Reference" "#PWR056"
+			(at 167.64 76.2 0)
+			(effects
+				(font
+					(size 1.27 1.27)
+				)
+				(hide yes)
+			)
+		)
+		(property "Value" "+3.3V"
+			(at 167.64 67.31 0)
+			(effects
+				(font
+					(size 1.27 1.27)
+				)
+			)
+		)
+		(property "Footprint" ""
+			(at 167.64 72.39 0)
+			(effects
+				(font
+					(size 1.27 1.27)
+				)
+				(hide yes)
+			)
+		)
+		(property "Datasheet" ""
+			(at 167.64 72.39 0)
+			(effects
+				(font
+					(size 1.27 1.27)
+				)
+				(hide yes)
+			)
+		)
+		(property "Description" "Power symbol creates a global label with name \"+3.3V\""
+			(at 167.64 72.39 0)
+			(effects
+				(font
+					(size 1.27 1.27)
+				)
+				(hide yes)
+			)
+		)
+		(pin "1"
+		)
+		(instances
+			(project "rulerSchematic"
+				(path "/a1545928-1195-40b9-b3c4-78f837012afb/494e6d32-1eab-4497-b57f-12dbcea47915"
+					(reference "#PWR056")
+					(unit 1)
+				)
+			)
+		)
+	)
+	(symbol
 		(lib_id "Device:C")
 		(at 133.35 135.89 0)
@@
 					(unit 1)
 				)
+			)
+		)
+	)
+	(symbol
+		(lib_id "power:+3.3V")
+		(at 213.36 123.19 0)
+		(unit 1)
+		(exclude_from_sim no)
+		(in_bom yes)
+		(on_board yes)
+		(dnp no)
+		(fields_autoplaced yes)
+		(property "Reference" "#PWR055"
+			(at 213.36 127 0)
+			(effects
+				(font
+					(size 1.27 1.27)
+				)
+				(hide yes)
+			)
+		)
+		(property "Value" "+3.3V"
+			(at 213.36 118.11 0)
+			(effects
+				(font
+					(size 1.27 1.27)
+				)
+			)
+		)
+		(property "Footprint" ""
+			(at 213.36 123.19 0)
+			(effects
+				(font
+					(size 1.27 1.27)
+				)
+				(hide yes)
+			)
+		)
+		(property "Datasheet" ""
+			(at 213.36 123.19 0)
+			(effects
+				(font
+					(size 1.27 1.27)
+				)
+				(hide yes)
+			)
+		)
+		(property "Description" "Power symbol creates a global label with name \"+3.3V\""
+			(at 213.36 123.19 0)
+			(effects
+				(font
+					(size 1.27 1.27)
+				)
+				(hide yes)
+			)
+		)
+		(pin "1"
+		)
+		(instances
+			(project "rulerSchematic"
+				(path "/a1545928-1195-40b9-b3c4-78f837012afb/494e6d32-1eab-4497-b57f-12dbcea47915"
+					(reference "#PWR055")
+					(unit 1)
+				)

Commit message: J'ai ajouter des power Flag pour spécifier a Kicad que c'est chill (faut qu'il apprenne a ce géré quand même)
Changed lines of the file:
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@@
+	)
+	(junction
+		(at 52.07 86.36)
+		(diameter 0)
+		(color 0 0 0 0)
 	)
 	(junction
@@
 		(pts
 			(xy 71.12 166.37) (xy 105.41 166.37)
+		)
+		(stroke
+			(width 0)
+			(type default)
+		)
+	)
+	(wire
+		(pts
+			(xy 43.18 86.36) (xy 52.07 86.36)
 		)
 		(stroke
@@
 					(unit 1)
 				)
+			)
+		)
+	)
+	(symbol
+		(lib_id "power:PWR_FLAG")
+		(at 43.18 86.36 90)
+		(unit 1)
+		(exclude_from_sim no)
+		(in_bom yes)
+		(on_board yes)
+		(dnp no)
+		(fields_autoplaced yes)
+		(property "Reference" "#FLG01"
+			(at 41.275 86.36 0)
+			(effects
+				(font
+					(size 1.27 1.27)
+				)
+				(hide yes)
+			)
+		)
+		(property "Value" "PWR_FLAG"
+			(at 39.37 86.3599 90)
+			(effects
+				(font
+					(size 1.27 1.27)
+				)
+				(justify left)
+			)
+		)
+		(property "Footprint" ""
+			(at 43.18 86.36 0)
+			(effects
+				(font
+					(size 1.27 1.27)
+				)
+				(hide yes)
+			)
+		)
+		(property "Datasheet" "~"
+			(at 43.18 86.36 0)
+			(effects
+				(font
+					(size 1.27 1.27)
+				)
+				(hide yes)
+			)
+		)
+		(property "Description" "Special symbol for telling ERC where power comes from"
+			(at 43.18 86.36 0)
+			(effects
+				(font
+					(size 1.27 1.27)
+				)
+				(hide yes)
+			)
+		)
+		(pin "1"
+		)
+		(instances
+			(project ""
+				(path "/a1545928-1195-40b9-b3c4-78f837012afb/494e6d32-1eab-4497-b57f-12dbcea47915"
+					(reference "#FLG01")
+					(unit 1)
+				)
