File: elec/Kicad/distanceSensor.kicad_sch (KiCad schematic)
At the start: 15 parts, among them J4 Conn_01x05, Q2 BSS138, Q3 BSS138, U5 VL53L0CXV0DH1, U6 MIC5219-2.8YM5

Commit message: add a few footprint
Parts:
- C10, C11, C12, C13, C15: footprint (none) -> Capacitor_SMD:C_0603_1608Metric_Pad1.08x0.95mm_HandSolder
- J4: footprint (none) -> Connector_PinSocket_2.54mm:PinSocket_1x05_P2.54mm_Vertical
- JP1: footprint (none) -> Jumper:SolderJumper-2_P1.3mm_Open_TrianglePad1.0x1.5mm
- R15, R16, R17: footprint (none) -> Resistor_SMD:R_0603_1608Metric_Pad0.98x0.95mm_HandSolder
- TP2: footprint (none) -> TestPoint:TestPoint_Loop_D1.80mm_Drill1.0mm_Beaded
Changed lines of the file:
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@@
 			)
 		)
-		(property "Footprint" ""
+		(property "Footprint" "Connector_PinSocket_2.54mm:PinSocket_1x05_P2.54mm_Vertical"
 			(at 95.25 152.4 0)
 			(effects
@@
 			)
 		)
-		(property "Footprint" ""
+		(property "Footprint" "Capacitor_SMD:C_0603_1608Metric_Pad1.08x0.95mm_HandSolder"
 			(at 194.0052 91.44 0)
 			(effects
@@
 			)
 		)
-		(property "Datasheet" "~"
+		(property "Datasheet" "https://www.digikey.ca/en/products/detail/yageo/CC0603KRX7R7BB104/302822"
 			(at 193.04 87.63 0)
 			(effects
@@
 			)
 		)
-		(property "Footprint" ""
+		(property "Footprint" "Resistor_SMD:R_0603_1608Metric_Pad0.98x0.95mm_HandSolder"
 			(at 56.388 59.69 90)
 			(effects
@@
 			)
 		)
-		(property "Footprint" ""
+		(property "Footprint" "TestPoint:TestPoint_Loop_D1.80mm_Drill1.0mm_Beaded"
 			(at 228.6 78.74 0)
 			(effects
@@
 			)
 		)
-		(property "Footprint" ""
+		(property "Footprint" "Resistor_SMD:R_0603_1608Metric_Pad0.98x0.95mm_HandSolder"
 			(at 48.768 59.69 90)
 			(effects
@@
 			)
 		)
-		(property "Footprint" ""
+		(property "Footprint" "Capacitor_SMD:C_0603_1608Metric_Pad1.08x0.95mm_HandSolder"
 			(at 154.6352 91.44 0)
 			(effects
@@
 			)
 		)
-		(property "Footprint" ""
+		(property "Footprint" "Capacitor_SMD:C_0603_1608Metric_Pad1.08x0.95mm_HandSolder"
 			(at 144.4752 91.44 0)
 			(effects
@@
 			)
 		)
-		(property "Datasheet" "~"
+		(property "Datasheet" "https://www.digikey.ca/en/products/detail/yageo/CC0603KRX7R7BB104/302822"
 			(at 143.51 87.63 0)
 			(effects
@@
 			)
 		)
-		(property "Footprint" ""
+		(property "Footprint" "Jumper:SolderJumper-2_P1.3mm_Open_TrianglePad1.0x1.5mm"
 			(at 105.41 81.28 0)
 			(effects
@@
 			)
 		)
-		(property "Footprint" ""
+		(property "Footprint" "Resistor_SMD:R_0603_1608Metric_Pad0.98x0.95mm_HandSolder"
 			(at 100.33 94.742 90)
 			(effects
@@
 			)
 		)
-		(property "Footprint" ""
+		(property "Footprint" "Capacitor_SMD:C_0603_1608Metric_Pad1.08x0.95mm_HandSolder"
 			(at 180.0352 91.44 0)
 			(effects
@@
 			)
 		)
-		(property "Footprint" ""
+		(property "Footprint" "Capacitor_SMD:C_0603_1608Metric_Pad1.08x0.95mm_HandSolder"
 			(at 229.5652 91.44 0)
 			(effects

Commit message: commencer le PCB vite fait
Parts:
- removed TP2: 2.8V, TestPoint:TestPoint_Loop_D1.80mm_Drill1.0mm_Beaded, symbol Connector:TestPoint
Changed lines of the file:
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@@
-	)
-	(junction
-		(at 223.52 82.55)
-		(diameter 0)
-		(color 0 0 0 0)
 	)
 	(junction
@@
 	(wire
 		(pts
-			(xy 223.52 82.55) (xy 228.6 82.55)
-		)
-		(stroke
-			(width 0)
-			(type default)
-		)
-	)
-	(wire
-		(pts
 			(xy 228.6 91.44) (xy 228.6 92.71)
 		)
@@
 	(wire
 		(pts
-			(xy 223.52 78.74) (xy 223.52 82.55)
-		)
-		(stroke
-			(width 0)
-			(type default)
-		)
-	)
-	(wire
-		(pts
 			(xy 69.85 67.31) (xy 82.55 67.31)
 		)
@@
 	(wire
 		(pts
-			(xy 218.44 82.55) (xy 223.52 82.55)
+			(xy 218.44 82.55) (xy 228.6 82.55)
 		)
 		(stroke
@@
 					(unit 1)
 				)
-			)
-		)
-	)
-	(symbol
-		(lib_id "Connector:TestPoint")
-		(at 223.52 78.74 0)
-		(unit 1)
-		(exclude_from_sim no)
-		(in_bom yes)
-		(on_board yes)
-		(dnp no)
-		(property "Reference" "TP2"
-			(at 221.996 70.612 0)
-			(effects
-				(font
-					(size 1.27 1.27)
-				)
-				(justify left)
-			)
-		)
-		(property "Value" "2.8V"
-			(at 221.488 72.898 0)
-			(effects
-				(font
-					(size 1.27 1.27)
-				)
-				(justify left)
-			)
-		)
-		(property "Footprint" "TestPoint:TestPoint_Loop_D1.80mm_Drill1.0mm_Beaded"
-			(at 228.6 78.74 0)
-			(effects
-				(font
-					(size 1.27 1.27)
-				)
-				(hide yes)
-			)
-		)
-		(property "Datasheet" "~"
-			(at 228.6 78.74 0)
-			(effects
-				(font
-					(size 1.27 1.27)
-				)
-				(hide yes)
-			)
-		)
-		(property "Description" "test point"
-			(at 223.52 78.74 0)
-			(effects
-				(font
-					(size 1.27 1.27)
-				)
-				(hide yes)
-			)
-		)
-		(pin "1"
-		)
-		(instances
-			(project "rulerSchematic"
-				(path "/a1545928-1195-40b9-b3c4-78f837012afb/5f7b9d88-eb12-47e8-8ae8-265c4903ec29"
-					(reference "TP2")
-					(unit 1)
-				)

Commit message: Jpense pas boire jeudi sérieux vue que y'a pas de 5@8
routage du découplage et des CLK
Parts:
- C10, C11, C12, C13, C15: footprint Capacitor_SMD:C_0603_1608Metric_Pad1.08x0.95mm_HandSolder -> Capacitor_SMD:C_0402_1005Metric_Pad0.74x0.62mm_HandSolder
- R15, R16, R17: footprint Resistor_SMD:R_0603_1608Metric_Pad0.98x0.95mm_HandSolder -> Resistor_SMD:R_0402_1005Metric_Pad0.72x0.64mm_HandSolder
Changed lines of the file:
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@@
 			)
 		)
-		(property "Footprint" "Capacitor_SMD:C_0603_1608Metric_Pad1.08x0.95mm_HandSolder"
+		(property "Footprint" "Capacitor_SMD:C_0402_1005Metric_Pad0.74x0.62mm_HandSolder"
 			(at 194.0052 91.44 0)
 			(effects
@@
 			)
 		)
-		(property "Footprint" "Resistor_SMD:R_0603_1608Metric_Pad0.98x0.95mm_HandSolder"
+		(property "Footprint" "Resistor_SMD:R_0402_1005Metric_Pad0.72x0.64mm_HandSolder"
 			(at 56.388 59.69 90)
 			(effects
@@
 			)
 		)
-		(property "Footprint" "Resistor_SMD:R_0603_1608Metric_Pad0.98x0.95mm_HandSolder"
+		(property "Footprint" "Resistor_SMD:R_0402_1005Metric_Pad0.72x0.64mm_HandSolder"
 			(at 48.768 59.69 90)
 			(effects
@@
 			)
 		)
-		(property "Footprint" "Capacitor_SMD:C_0603_1608Metric_Pad1.08x0.95mm_HandSolder"
+		(property "Footprint" "Capacitor_SMD:C_0402_1005Metric_Pad0.74x0.62mm_HandSolder"
 			(at 154.6352 91.44 0)
 			(effects
@@
 			)
 		)
-		(property "Footprint" "Capacitor_SMD:C_0603_1608Metric_Pad1.08x0.95mm_HandSolder"
+		(property "Footprint" "Capacitor_SMD:C_0402_1005Metric_Pad0.74x0.62mm_HandSolder"
 			(at 144.4752 91.44 0)
 			(effects
@@
 			)
 		)
-		(property "Footprint" "Resistor_SMD:R_0603_1608Metric_Pad0.98x0.95mm_HandSolder"
+		(property "Footprint" "Resistor_SMD:R_0402_1005Metric_Pad0.72x0.64mm_HandSolder"
 			(at 100.33 94.742 90)
 			(effects
@@
 			)
 		)
-		(property "Footprint" "Capacitor_SMD:C_0603_1608Metric_Pad1.08x0.95mm_HandSolder"
+		(property "Footprint" "Capacitor_SMD:C_0402_1005Metric_Pad0.74x0.62mm_HandSolder"
 			(at 180.0352 91.44 0)
 			(effects
@@
 			)
 		)
-		(property "Footprint" "Capacitor_SMD:C_0603_1608Metric_Pad1.08x0.95mm_HandSolder"
+		(property "Footprint" "Capacitor_SMD:C_0402_1005Metric_Pad0.74x0.62mm_HandSolder"
 			(at 229.5652 91.44 0)
 			(effects

Commit message: abdel aziz clutch l'app5
Parts:
- removed J4: Conn_01x05, Connector_PinSocket_2.54mm:PinSocket_1x05_P2.54mm_Vertical, symbol Connector_Generic:Conn_01x05
- removed JP1: SolderJumper_2_Open, Jumper:SolderJumper-2_P1.3mm_Open_TrianglePad1.0x1.5mm, symbol Jumper:SolderJumper_2_Open
- added J10: Conn_01x06, Connector_PinSocket_2.54mm:PinSocket_1x06_P2.54mm_Vertical, symbol Connector_Generic:Conn_01x06
- added J4: Conn_01x06, Connector_PinHeader_2.54mm:PinHeader_1x06_P2.54mm_Horizontal, symbol Connector_Generic:Conn_01x06
- added R19, R20: 10K, Resistor_SMD:R_0402_1005Metric_Pad0.72x0.64mm_HandSolder, symbol Device:R
- added R32: Bypass_XSHUT (0 ohm), Resistor_SMD:R_0402_1005Metric_Pad0.72x0.64mm_HandSolder, symbol Device:R
Connections:
- net +2V8: now also J10.2 (Pin_2), J4.2 (Pin_2), R32.2
- net +3.3V: now also J10.1 (Pin_1), J4.1 (Pin_1), R19.1, R20.1
- net GND: now also J10.6 (Pin_6), J4.6 (Pin_6)
- net I2C1_SCL: now also J10.4 (Pin_4), J4.4 (Pin_4), R19.2
- net I2C1_SDA: now also J10.3 (Pin_3), J4.3 (Pin_3), R20.2
- net XSHUT: now also J10.5 (Pin_5), J4.5 (Pin_5)
- net at R17.2, U5.5 (XSHUT): now also R32.1
Other:
- moved on the sheet: Q2, Q3, R15, R16

Commit message: j'essaye de fix la hauteur des designator pis si sa scrap cv être ça
Parts:
- J10: value Conn_01x06 -> TouillomètreMount
- J4: value Conn_01x06 -> ToFMount
Connections:
- net +3.3V: no longer C12.1, C15.1, J4.1 (Pin_1), R19.1, R20.1, U6.1 (IN), U6.3 (EN)
- net I2C1_SCL: no longer J4.4 (Pin_4), Q3.3 (D), R19.2
- net I2C1_SDA: no longer J4.3 (Pin_3), Q2.3 (D), R20.2
- net XSHUT: no longer J4.5 (Pin_5), R17.1
- new net +3V3: C12.1, C15.1, J4.1 (Pin_1), R19.1, R20.1, U6.1 (IN), U6.3 (EN)
- new net I2C_SCL: J4.4 (Pin_4), Q3.3 (D), R19.2
- new net I2C_SDA: J4.3 (Pin_3), Q2.3 (D), R20.2
- new net XSHUT_Breakout: J4.5 (Pin_5), R17.1
Other:
- note added: "Sur le Touillomètre"
- moved on the sheet: J10, J4

Commit message: jpense qu'on est ready to order
Connections:
- net +3V3 is gone; now on net +3.3V: C12.1, C15.1, J4.1 (Pin_1), R19.1, R20.1, U6.1 (IN), U6.3 (EN)

Commit message: généré la schematic
Other:
- note added: "Permet de transformer la logique SDA/SCL qui est de 3.3V a une logique SDA/SCL de 2.8V"
- note added: "Petit LDO (Low Drop Regulator) 3V3 ---> 2V8"
- note added: "XSHUT = peremet de désactiver le capteur en mettant cette broche a LOW."
- note removed: "GPIO1 est une sortie qui permet de trigg des interrupt ex: distance aillant atteint un seuil prédéfini options: 1. soit on le connecte pour avoir des notifs 2. on le connect pas (présentement pas connecté)"
- note removed: "Magouille pour transformer la logique SDA/SCL qui est de 3.3V a une logique SDA/SCL de 2.8V Trust it should work (In JULIEN we Trust)"
- note removed: "XSHUT = peremet de désactiver le capteur en mettant cette broche a LOW. Il ne consommera pas bcp d'énergie a ce momment là options: 1. soit on le met a high (2.8V) 2. on le connecte au MCU et qu'on le met a high quand on veux l'utiliser (présentement connecté)"
- company: (none) -> University of Sherbrooke
- title: (none) -> Touillometre - ToF Distance Sensor
Changed lines of the file:
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@@
 	(generator_version "8.0")
 	(paper "A4")
+	(title_block
+		(title "Touillometre - ToF Distance Sensor")
+		(date "2024-12-26")
+		(rev "C3I")
+		(company "University of Sherbrooke")
+	)
 	(junction
 		(at 52.07 81.28)
@@
 		)
 	)
-	(text "Magouille pour transformer la logique SDA/SCL qui est de 3.3V a une logique SDA/SCL de 2.8V \nTrust it should work (In JULIEN we Trust)"
+	(text "Permet de transformer la logique SDA/SCL qui est de 3.3V a une logique SDA/SCL de 2.8V "
 		(exclude_from_sim no)
 		(at 72.39 35.306 0)
@@
 		)
 	)
-	(text "GPIO1 est une sortie qui permet de trigg des interrupt\nex: distance aillant atteint un seuil prédéfini\noptions: 1. soit on le connecte pour avoir des notifs\n2. on le connect pas (présentement pas connecté)\n\n"
+	(text "Petit LDO (Low Drop Regulator) 3V3 ---> 2V8"
 		(exclude_from_sim no)
-		(at 131.064 129.794 0)
+		(at 205.74 70.612 0)
 		(effects
 			(font
@@
 	(text "Ceci est un petit PCB\non veux pouvoir le retirer et le remettre avec un header"
 		(exclude_from_sim no)
-		(at 56.896 24.384 0)
+		(at 64.008 23.876 0)
 		(effects
 			(font
 				(size 1.778 1.778)
+				(thickness 0.3556)
+				(bold yes)
 				(italic yes)
 			)
@@
 		)
 	)
-	(text "XSHUT = peremet de désactiver le capteur\nen mettant cette broche a LOW.\nIl ne consommera pas bcp d'énergie a ce momment là\noptions: 1. soit on le met a high (2.8V)\n2. on le connecte au MCU et qu'on le met a high quand on veux l'utiliser (présentement connecté)\n"
+	(text "XSHUT = peremet de désactiver le capteur\nen mettant cette broche a LOW.\n"
 		(exclude_from_sim no)
-		(at 133.604 117.348 0)
+		(at 128.524 116.078 0)
 		(effects
 			(font
