File: elec/Kicad/rulerSchematic.kicad_pcb (KiCad board)
At the start: 2 copper layers, 113 parts, among them J1 USART, J2 B2B-XH-A, J3 HX0201800000G, J4 Conn_01x05, J5 TestPoint, J6 SWD, J7 USB_B_Micro_MAIN, J8 SD_CARD_CONN, J9 Conn_01x13, Q1 SI2323DS-T1, Q2 BSS138, Q3 BSS138, Q4 SS8050, Q5 NTK3043NT1G, SW1 SW_Push_Gauche_GO_IN, SW2 SW_Push_Droite_GO_BACK, SW3 SW_Push_Action_LOG_EXIT, SW5 SW_Push_BOOT, SW6 SW_Push_RESET, U1 STM32L053C8T6, U11 MMC5633NJL, U2 BMI160, U3 MCP73831, U4 HTU21D, U5 VL53L0CXV0DH1, U6 MIC5219-2.8YM5, U8 LTR-303ALS-01, U9 TLV62085RLTR, Y1 32MHz, Y2 32.768KHz

Commit message: touillerie
Parts:
- removed SW6: SW_Push_RESET, Button_Switch_SMD:SW_SPST_PTS647_Sx38
- added C5: 100nF, Capacitor_SMD:C_0603_1608Metric_Pad1.08x0.95mm_HandSolder, F.Cu at (66.5, 163.1)
- added F2: F0603G0R03FNTR, F0603G0R03FNTR:F0603G0R03FNTR, F.Cu at (57.0, 160.1)
- added SW4: SW_Push_RESET, B3U_1100P:B3U-1100P_OMR, F.Cu at (70.0, 35.7)
- J1, J6: footprint Connector_PinHeader_2.54mm:PinHeader_1x04_P2.54mm_Vertical -> Connector_PinHeader_2.54mm:PinHeader_1x02_P2.54mm_Vertical
- SW1, SW2, SW3: footprint Button_Switch_SMD:SW_SPST_PTS645 -> tacticleSwitch4_5x4_5mm:SWITCH_TR2LFS
- SW5: footprint Button_Switch_SMD:SW_SPST_PTS647_Sx38 -> B3U_1100P:B3U-1100P_OMR
- moved C22 201.0 mm to (66.5, 157.5), turned to 0 degrees
- moved U11 193.6 mm to (70.1, 154.8)
- moved F1 84.8 mm to (56.9, 155.1), turned to 90 degrees
- moved U4 83.7 mm to (65.0, 76.1)
- moved R22 80.4 mm to (60.8, 159.0), turned to 90 degrees
- moved C9 79.7 mm to (59.3, 76.1)
- moved R24 78.0 mm to (62.9, 158.9), turned to 90 degrees
- moved D6 74.3 mm to (66.2, 160.6)
- moved D4 73.6 mm to (70.2, 158.9), turned to 90 degrees
- moved J1 53.8 mm to (75.1, 84.8)
- moved J5 52.9 mm to (75.1, 57.6)
- moved C21 49.0 mm to (69.9, 105.9)
- moved U8 45.6 mm to (66.3, 105.9)
- moved S1 29.0 mm to (74.8, 43.2), turned to -90 degrees
- moved C20 19.2 mm to (66.5, 155.5)
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Connections:
- C25 pad 1: Vbat -> Vin
- C34 pad 2: Net-(U9-PG) -> GND
- D4 pad C: GND -> Net-(C5-Pad2)
- D6 pad K: GND -> Net-(D4-PadA)
- J1 pad 1: +3.3V -> USART1_TX
- J1 pad 2: USART1_TX -> USART1_RX
- J3 pad 1: unconnected-(J3-Pad1) -> Net-(J3-Pad1)
- J3 pad 2: Net-(J3-Pad2) -> Net-(J3-Pad1)
- J3 pad 3: unconnected-(J3-Pad3) -> Net-(D4-PadA)
- J6 pad 1: +3.3V -> SWDIO
- J6 pad 2: SWDIO -> SWCLK
- R24 pad 2: Net-(J3-Pad2) -> Net-(J3-Pad1)
- R31 pad 2: Net-(U9-PG) -> GND
- R4 pad 1: Vbat -> Vin
- R6 pad 1: Vbat -> Vin
- S1 pad 1B: Vbat -> Vin
- SW1 pad 1: +3.3V -> PB11_Bouton_IN
- SW1 pad 2: PB11_Bouton_IN -> unconnected-(SW1-Pad2)
- SW2 pad 1: +3.3V -> PB10_Bouton_BACK
- SW2 pad 2: PB10_Bouton_BACK -> unconnected-(SW2-Pad2)
- SW3 pad 1: +3.3V -> PB2_Bouton_LOG
- SW3 pad 2: PB2_Bouton_LOG -> unconnected-(SW3-Pad2)
- SW5 pad 1: +3.3V -> BOOT0
- SW5 pad 2: BOOT0 -> +3.3V
- U1 pad 18: read_pin_high -> read_pin
- U1 pad 19: read_pin_low -> unconnected-(U1-PB1-Pad19)
- U9 pad 1: Vbat -> Vin
- U9 pad 7: Vbat -> Vin
Other:
- board text added: "U4"
- board text removed: "Changer le sensor"
- board text removed: "Magouille a charles"

Commit message: igfukhj.hlk
Parts:
- added H1: MountingHole, MountingHole:MountingHole_2.2mm_M2, F.Cu at (56.8, 133.5)
- added H2: MountingHole, MountingHole:MountingHole_2.2mm_M2, F.Cu at (70.5, 133.5)
- added H3: MountingHole, MountingHole:MountingHole_2.2mm_M2, F.Cu at (56.8, 161.2)
- added H4: MountingHole, MountingHole:MountingHole_2.2mm_M2, F.Cu at (70.5, 161.2)
- moved R8 85.5 mm to (56.5, 46.6), turned to 0 degrees
- moved R9 80.2 mm to (61.4, 49.5), turned to 90 degrees
- moved C6 80.1 mm to (63.6, 49.5)
- moved C4 79.9 mm to (54.1, 49.8), turned to -90 degrees
- moved U3 79.7 mm to (57.8, 49.5), turned to 180 degrees
- moved D3 72.6 mm to (53.1, 46.5), turned to 180 degrees
- moved U11 18.9 mm to (54.3, 165.2)
- moved JP4 17.3 mm to (40.2, 36.4)
- moved JP2 17.3 mm to (40.3, 40.6)
- moved C36 16.0 mm to (55.0, 116.6)
- moved R36 16.0 mm to (55.0, 119.0)
- moved R37 16.0 mm to (55.0, 121.6)
- moved R38 16.0 mm to (55.0, 124.0)
- moved R39 16.0 mm to (55.0, 126.5)
- moved C22 11.4 mm to (58.6, 165.8)
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Other:
- board outline added: 30.1 x 155.6 mm

Commit message: Jpense pas boire jeudi sérieux vue que y'a pas de 5@8
routage du découplage et des CLK
Parts:
- added R12: 10K, Resistor_SMD:R_0402_1005Metric_Pad0.72x0.64mm_HandSolder, F.Cu at (72.8, 59.4)
- added R7: 10K, Resistor_SMD:R_0402_1005Metric_Pad0.72x0.64mm_HandSolder, F.Cu at (72.8, 61.8)
- C1, C10, C11, C12, C13, C14, C15, C16, C17, C18, C19, C2, C20, C21, C22, C23, C24, C25, C26, C27, C28, C29, C3, C30, C31, C32, C33, C34, C35, C36, C4, C5, C6, C7, C8, C9: footprint Capacitor_SMD:C_0603_1608Metric_Pad1.08x0.95mm_HandSolder -> Capacitor_SMD:C_0402_1005Metric_Pad0.74x0.62mm_HandSolder
- J2: footprint Connector_JST:JST_XH_B2B-XH-AM_1x02_P2.50mm_Vertical -> Connector_JST:JST_XH_S2B-XH-A_1x02_P2.50mm_Horizontal
- R1, R10, R11, R13, R14, R15, R16, R17, R19, R2, R20, R21, R22, R23, R24, R25, R26, R27, R28, R29, R3, R30, R31, R36, R37, R38, R39, R4, R5, R6, R8, R9: footprint Resistor_SMD:R_0603_1608Metric_Pad0.98x0.95mm_HandSolder -> Resistor_SMD:R_0402_1005Metric_Pad0.72x0.64mm_HandSolder
- moved C26 17.0 mm to (70.8, 65.8), turned to -135 degrees
- moved JP3 14.7 mm to (39.6, 104.5)
- moved R3 13.0 mm to (63.6, 111.7), turned to 90 degrees
- moved C17 12.7 mm to (52.6, 62.0), turned to 90 degrees
- moved C29 10.2 mm to (56.8, 58.6), turned to 45 degrees
- moved Y2 9.84 mm to (54.4, 62.1), turned to -90 degrees
- moved D2 8.76 mm to (61.8, 107.8)
- moved J2 7.83 mm to (68.3, 103.8), turned to 0 degrees
- moved C18 7.74 mm to (56.2, 61.9), turned to -90 degrees
- moved C21 6.77 mm to (63.2, 104.9)
- moved U8 5.92 mm to (60.4, 105.4)
- moved R5 4.90 mm to (57.6, 105.5)
- moved R6 4.52 mm to (55.0, 101.9)
- moved R14 4.50 mm to (55.0, 105.7)
- moved Q5 4.39 mm to (57.6, 102.4)
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Connections:
- SW4 pad 1: NRST -> GND
- SW4 pad 2: GND -> NRST
- U1 pad 10: unconnected-(U1-PA0-Pad10) -> CS_LCD
- U1 pad 19: unconnected-(U1-PB1-Pad19) -> RS_LCD
- U1 pad 26: CS_LCD -> I2C1_SCL
- U1 pad 27: unconnected-(U1-PB14-Pad27) -> I2C1_SDA
- U1 pad 28: unconnected-(U1-PB15-Pad28) -> XSHUT
- U1 pad 40: RS_LCD -> unconnected-(U1-PB4-Pad40)
- U1 pad 41: XSHUT -> unconnected-(U1-PB5-Pad41)
- U1 pad 45: I2C1_SCL -> unconnected-(U1-PB8-Pad45)
- U1 pad 46: I2C1_SDA -> unconnected-(U1-PB9-Pad46)
Routing:
- net GND: track 0.00 -> 27.3 mm, vias 0 -> 7
- net +3.3V: track 0.00 -> 10.2 mm
- net OSC_OUT: track 0.00 -> 9.23 mm
- net OSC32_OUT: track 0.00 -> 8.80 mm
- net OSC32_IN: track 0.00 -> 7.94 mm
- net OSC_IN: track 0.00 -> 6.02 mm
- net +3.3VA: track 0.00 -> 4.28 mm
- added copper zone on B.Cu, net GND
Other:
- board size 30.1 x 155.6 mm -> 30.1 x 155 mm
- board text added: "Changer le connecteur de la batterie pour le :S2B-XH-A-1"

Commit message: bloatware
fait le slikscree de mesure (merci jabooby)
Other:
- board text added: "0"
- board text added: "1"
- board text added: "10"
- board text added: "11"
- board text added: "12"
- board text added: "13"
- board text added: "14"
- board text added: "15"
- board text added: "2"
- board text added: "3"
- board text added: "4"
- board text added: "5"
- board text added: "6"
- board text added: "7"
- board text added: "8"
- board text added: "9"

Commit message: sorry Jacob tu va être dessus ...
Parts:
- removed J4: Conn_01x05, Connector_PinSocket_2.54mm:PinSocket_1x05_P2.54mm_Vertical
- removed R19, R20: 10K, Resistor_SMD:R_0402_1005Metric_Pad0.72x0.64mm_HandSolder
- added J10: mount_touillometre, Connector_PinSocket_2.54mm:PinSocket_1x06_P2.54mm_Vertical, F.Cu at (59.2, 185.6)
- added J11: mount_protoBoard, Connector_PinSocket_2.54mm:PinSocket_1x06_P2.54mm_Vertical, F.Cu at (99.1, 176.8)
- J2, JP2, JP3, JP4: moved to B.Cu
- moved C10 192.3 mm to (112.8, 180.4)
- moved C11 192.3 mm to (112.8, 183.2)
- moved C12 192.3 mm to (113.0, 186.2)
- moved C13 192.3 mm to (113.0, 188.7)
- moved C15 192.3 mm to (113.0, 191.2)
- moved JP1 192.3 mm to (117.5, 179.8)
- moved Q2 192.3 mm to (126.2, 178.0)
- moved Q3 192.3 mm to (126.2, 182.7)
- moved R15 192.3 mm to (117.4, 183.5)
- moved R16 192.3 mm to (117.4, 186.0)
- moved R17 192.3 mm to (117.5, 189.4)
- moved U5 192.3 mm to (105.9, 181.8)
- moved U6 192.3 mm to (127.5, 190.4)
- moved JP3 58.7 mm to (71.7, 55.3)
- moved R5 55.4 mm to (72.2, 52.0)
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Connections:
- C9 pad 2: Net-(C9-Pad2) -> GND
- U1 pad 2: unconnected-(U1-PC13-Pad2) -> RESET_LCD
- U1 pad 21: PB10_Bouton_BACK -> PB11_Bouton_IN
- U1 pad 22: PB11_Bouton_IN -> PB10_Bouton_BACK
- U1 pad 39: RESET_LCD -> unconnected-(U1-PB3-Pad39)
- U4 pad 2: Net-(C9-Pad2) -> GND
- U4 pad PAD: Net-(C9-Pad2) -> GND
Routing:
- net +3.3V: track 10.2 -> 242.0 mm, vias 0 -> 9
- net +2V8: track 0.00 -> 135.6 mm, vias 0 -> 1
- net read_pin: track 0.00 -> 104.6 mm, vias 0 -> 2
- net I2C1_SDA: track 0.00 -> 78.8 mm, vias 0 -> 3
- net I2C1_SCL: track 0.00 -> 77.5 mm, vias 0 -> 3
- net GND: track 27.3 -> 98.4 mm, vias 7 -> 25
- net RESET_LCD: track 0.00 -> 66.7 mm, vias 0 -> 2
- net RS_LCD: track 0.00 -> 63.0 mm, vias 0 -> 2
- net NRST: track 0.00 -> 59.0 mm
- net PB2_Bouton_LOG: track 0.00 -> 58.8 mm, vias 0 -> 2
- net BL_LCD: track 0.00 -> 54.6 mm, vias 0 -> 2
- net +5V: track 0.00 -> 45.7 mm, vias 0 -> 2
- net BAT_PERCENT: track 0.00 -> 42.7 mm, vias 0 -> 3
- net BOOT0: track 0.00 -> 34.4 mm, vias 0 -> 4
- net PB11_Bouton_IN: track 0.00 -> 30.1 mm
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Other:
- board text added: "Rajouter un 2.8V ici (ou enlever celui en haut)"
- board text removed: "U4"
