File: elec/Kicad/rulerSchematic.kicad_pcb (KiCad board)
At the start: 2 copper layers, 30.1 x 173.7 mm, 119 parts, among them J1 USART, J10 TouillomètreMount, J2 S2B-XH-A, J3 HX0201800000G, J4 ToFMount, J5 TestPoint, J6 SWD, J7 USB_B_Micro_MAIN, J8 SD_CARD_CONN, J9 Conn_01x13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

Commit message: je vais au costco tantot i guess que c'est chill
Routing:
- net GND: track 98.5 -> 104.5 mm, vias 80 -> 332

Commit message: dd
Routing:
- net GND: vias 332 -> 330
Changed lines of the file:
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@@
 		(tags "Fuse")
 		(property "Reference" "F2"
-			(at 1.2 -2.1 90)
+			(at 1.144998 -2.459231 90)
 			(layer "F.SilkS")
 			(effects
@@
 		(at 146.806731 125.324998 -90)
 		(property "Reference" "J8"
-			(at 6.8 -9.3125 90)
+			(at 6.675002 -9.393269 90)
 			(layer "F.SilkS")
 			(effects
@@
 		(tags "resistor handsolder")
 		(property "Reference" "R24"
-			(at 0.0125 1.12 0)
+			(at -0.778269 1.12 0)
 			(layer "F.SilkS")
 			(effects
@@
 		(tags "capacitor handsolder")
 		(property "Reference" "C20"
-			(at -0.0675 1 90)
+			(at -0.0675 0.869231 90)
 			(layer "F.SilkS")
 			(effects
@@
 		(tags "Connector")
 		(property "Reference" "J3"
-			(at 2.3 -5.15 90)
+			(at -2.525002 0.780769 180)
 			(layer "F.SilkS")
 			(effects
@@
 		(tags "resistor handsolder")
 		(property "Reference" "R1"
-			(at -0.929231 -0.894998 0)
+			(at -1.729231 0.005002 90)
 			(layer "F.SilkS")
 			(effects
@@
 		(at 150.156731 147.344998)
 		(property "Reference" "D4"
-			(at 3.01 -0.25 90)
+			(at 2.843269 -1.144998 90)
 			(layer "F.SilkS")
 			(effects
@@
 		(tags "capacitor handsolder")
 		(property "Reference" "C26"
-			(at -0.141421 -0.989949 -135)
+			(at -0.594605 -1.03555 -135)
 			(layer "F.SilkS")
 			(effects
@@
 	)
 	(gr_text "3V3\n"
-		(at 143.3 162.8 180)
+		(at 143.2 163 180)
 		(layer "F.SilkS")
 		(effects
@@
 	)
 	(gr_text "13"
-		(at 161.492948 33.174998 -90)
+		(at 161.492948 33.174998 270)
 		(layer "F.SilkS")
 		(effects
@@
 	)
 	(via
-		(at 161.725 34.674998)
-		(size 0.8)
-		(drill 0.4)
-		(layers "F.Cu" "B.Cu")
-		(free yes)
-		(net 2)
-	)
-	(via
 		(at 162.2 58.2)
 		(size 0.8)
@@
 	)
 	(via
-		(at 161.725 24.674998)
-		(size 0.8)
-		(drill 0.4)
-		(layers "F.Cu" "B.Cu")
-		(free yes)
-		(net 2)
-	)
-	(via
 		(at 151.769231 38.199998)
 		(size 0.8)
@@
 	)
 	(via
-		(at 143.725 162.674998)
+		(at 144.4 162.6)
 		(size 0.8)
 		(drill 0.4)
@@
 			"28a57f69-8e9f-4c0c-858a-343fda586010" "28be8a9a-b941-4c86-9b34-153483fe3d1b"
 			"29632806-6dad-46e2-a2f4-4ab1ae1dcb87" "2a15199b-6675-4a8f-8721-d09e9435b8a2"
-			"2b0c24ea-1b70-4f50-a896-91534e8eaa7c" "2db1cefb-1438-4284-b6ae-8968514c4147"
-			"2f5a50f3-e942-4cb7-a782-ae3d3610a87a" "2fc1aee2-7ac1-4467-8422-0b3a81486bd5"
-			"2fd7409d-57f6-4cad-bb14-840142edfa02" "2feb065e-fd54-48b4-b183-38d6f14a1781"
+			"2db1cefb-1438-4284-b6ae-8968514c4147" "2f5a50f3-e942-4cb7-a782-ae3d3610a87a"
+			"2fc1aee2-7ac1-4467-8422-0b3a81486bd5" "2fd7409d-57f6-4cad-bb14-840142edfa02"
 			"3194fe0d-54d2-437d-99d6-4886b0a1e745" "31d9df68-de89-48ae-a60b-fde370dbf08f"
 			"330b3faa-df84-4bb8-b2fe-bc6ca4d205ee" "33cbaa18-2934-4f00-aa2b-f6a154d305c8"

Commit message: jpense qu'on est ready to order
Parts:
- added G***: LOGO, LOGO, B.Cu at (148.2, 70.5)
- moved C3 3.32 mm to (137.5, 49.5), turned to 90 degrees
- moved L1 2.95 mm to (139.2, 52.0)
Connections:
- C12 pad 1: +3V3 -> +3.3V
- C15 pad 1: +3V3 -> +3.3V
- C9 pad 2: Net-(C9-Pad2) -> GND
- J4 pad 1: +3V3 -> +3.3V
- R19 pad 1: +3V3 -> +3.3V
- R20 pad 1: +3V3 -> +3.3V
- U4 pad 2: Net-(C9-Pad2) -> GND
- U4 pad PAD: Net-(C9-Pad2) -> GND
- U6 pad 1: +3V3 -> +3.3V
- U6 pad 3: +3V3 -> +3.3V
Routing:
- net +3V3: track 27.5 -> 0.00 mm
- net +3.3V: track 512.9 -> 539.0 mm, vias 6 -> 5
- net Net-(C9-Pad2): track 3.55 -> 0.00 mm
- net GND: track 104.5 -> 108.0 mm, vias 330 -> 251
- net +3.3VA: track 6.13 -> 9.07 mm
- net XSHUT: track 137.0 -> 135.3 mm
Other:
- board text removed: "Acheter un Stencil"

Commit message: generated gerber files
Parts:
- moved R1 0.28 mm to (140.7, 54.1)
Routing:
- net BL_LCD: track 67.9 -> 70.1 mm
- net +3.3V: track 539.0 -> 537.3 mm
- net JOYSTICK_Y: track 45.3 -> 44.1 mm, vias 0 -> 2
- net JOYSTICK_X: track 43.9 -> 42.9 mm, vias 0 -> 2
- net GND: track 108.0 -> 107.9 mm, vias 251 -> 260

Commit message: gruiter
Routing:
- net GND: track 107.9 -> 106.0 mm, vias 260 -> 275
- net +5V: track 33.2 -> 33.7 mm
