File: elec/Kicad/temperatureHumiditySensor.kicad_sch (KiCad schematic)
At the start: 2 parts, among them U4 HTU21D

Commit message: jpense qu'on est ready to order
Connections:
- net GND: now reaches C9.2, U4.2 (GND), U4.PAD (GND)
Other:
- note removed: "Mettre des pull-up resistor sur la ligne I2C dans la schématique du MCU (Fait)"
Changed lines of the file:
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@@
+		(color 0 0 0 0)
+	)
+	(junction
+		(at 118.11 87.63)
+		(diameter 0)
 		(color 0 0 0 0)
 	)
@@
 		(exclude_from_sim no)
 		(at 135.382 39.116 0)
-		(effects
-			(font
-				(size 1.27 1.27)
-			)
-		)
-	)
-	(text "Mettre des pull-up resistor sur la ligne I2C dans la schématique du MCU (Fait)\n"
-		(exclude_from_sim no)
-		(at 176.53 35.306 0)
 		(effects
 			(font
@@
 					(unit 1)
 				)
+			)
+		)
+	)
+	(symbol
+		(lib_id "power:GND")
+		(at 118.11 87.63 0)
+		(unit 1)
+		(exclude_from_sim no)
+		(in_bom yes)
+		(on_board yes)
+		(dnp no)
+		(fields_autoplaced yes)
+		(property "Reference" "#PWR069"
+			(at 118.11 93.98 0)
+			(effects
+				(font
+					(size 1.27 1.27)
+				)
+				(hide yes)
+			)
+		)
+		(property "Value" "GND"
+			(at 118.11 92.71 0)
+			(effects
+				(font
+					(size 1.27 1.27)
+				)
+			)
+		)
+		(property "Footprint" ""
+			(at 118.11 87.63 0)
+			(effects
+				(font
+					(size 1.27 1.27)
+				)
+				(hide yes)
+			)
+		)
+		(property "Datasheet" ""
+			(at 118.11 87.63 0)
+			(effects
+				(font
+					(size 1.27 1.27)
+				)
+				(hide yes)
+			)
+		)
+		(property "Description" "Power symbol creates a global label with name \"GND\" , ground"
+			(at 118.11 87.63 0)
+			(effects
+				(font
+					(size 1.27 1.27)
+				)
+				(hide yes)
+			)
+		)
+		(pin "1"
+		)
+		(instances
+			(project ""
+				(path "/a1545928-1195-40b9-b3c4-78f837012afb/4cc0ebdd-0f2a-405e-9a30-83f437855272"
+					(reference "#PWR069")
+					(unit 1)
+				)
