File: elec/Kicad/temperatureHumiditySensor.kicad_sch (KiCad schematic)
At the start: 2 parts, among them U4 HTU21D

Commit message: généré la schematic
Other:
- company: (none) -> University of Sherbrooke
- title: (none) -> Touillomètre - Humidity Sensor
Changed lines of the file:
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@@
 	(generator_version "8.0")
 	(paper "A4")
+	(title_block
+		(title "Touillomètre - Humidity Sensor")
+		(date "2024-12-26")
+		(rev "C3I")
+		(company "University of Sherbrooke")
+	)
 	(junction
 		(at 118.11 59.69)
@@
 	(text "I2C address=0x40"
 		(exclude_from_sim no)
-		(at 135.382 39.116 0)
+		(at 137.922 47.244 0)
 		(effects
 			(font
