File: elec/Kicad/BatteryCharger.kicad_sch (KiCad schematic)
At the start: 11 parts, among them J2 B2B-XH-A, U3 MCP73831

Commit message: Jpense pas boire jeudi sérieux vue que y'a pas de 5@8
routage du découplage et des CLK
Parts:
- C4, C6: footprint Capacitor_SMD:C_0603_1608Metric_Pad1.08x0.95mm_HandSolder -> Capacitor_SMD:C_0402_1005Metric_Pad0.74x0.62mm_HandSolder
- J2: footprint Connector_JST:JST_XH_B2B-XH-AM_1x02_P2.50mm_Vertical -> Connector_JST:JST_XH_S2B-XH-A_1x02_P2.50mm_Horizontal
- R8, R9: footprint Resistor_SMD:R_0603_1608Metric_Pad0.98x0.95mm_HandSolder -> Resistor_SMD:R_0402_1005Metric_Pad0.72x0.64mm_HandSolder
Changed lines of the file:
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@@
 			)
 		)
-		(property "Footprint" "Connector_JST:JST_XH_B2B-XH-AM_1x02_P2.50mm_Vertical"
+		(property "Footprint" "Connector_JST:JST_XH_S2B-XH-A_1x02_P2.50mm_Horizontal"
 			(at 144.78 64.77 0)
 			(effects
@@
 			)
 		)
-		(property "Footprint" "Capacitor_SMD:C_0603_1608Metric_Pad1.08x0.95mm_HandSolder"
+		(property "Footprint" "Capacitor_SMD:C_0402_1005Metric_Pad0.74x0.62mm_HandSolder"
 			(at 125.4252 73.66 0)
 			(effects
@@
 			)
 		)
-		(property "Footprint" "Capacitor_SMD:C_0603_1608Metric_Pad1.08x0.95mm_HandSolder"
+		(property "Footprint" "Capacitor_SMD:C_0402_1005Metric_Pad0.74x0.62mm_HandSolder"
 			(at 65.7352 63.5 0)
 			(effects
@@
 			)
 		)
-		(property "Footprint" "Resistor_SMD:R_0603_1608Metric_Pad0.98x0.95mm_HandSolder"
+		(property "Footprint" "Resistor_SMD:R_0402_1005Metric_Pad0.72x0.64mm_HandSolder"
 			(at 113.792 71.12 90)
 			(effects
@@
 			)
 		)
-		(property "Footprint" "Resistor_SMD:R_0603_1608Metric_Pad0.98x0.95mm_HandSolder"
+		(property "Footprint" "Resistor_SMD:R_0402_1005Metric_Pad0.72x0.64mm_HandSolder"
 			(at 79.502 68.58 90)
 			(effects

Commit message: abdel aziz clutch l'app5
Parts:
- J2: value B2B-XH-A -> S2B-XH-A
Changed lines of the file:
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@@
 			)
 		)
-		(property "Value" "B2B-XH-A"
+		(property "Value" "S2B-XH-A"
 			(at 149.86 64.7701 0)
 			(effects

Commit message: généré la schematic
Other:
- note removed: "Valider si j'ai pas inverser les connexion ici du connecteur de la batterie"
- company: (none) -> University of Sherbrooke
- title: (none) -> Touillomètre - Battery Management
- moved on the sheet: H1, H2, H3, H4
Changed lines of the file:
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@@
 	(generator_version "8.0")
 	(paper "A4")
+	(title_block
+		(title "Touillomètre - Battery Management")
+		(date "2024-12-26")
+		(rev "C3I")
+		(company "University of Sherbrooke")
+	)
 	(junction
 		(at 124.46 80.01)
@@
 	)
 	(rectangle
-		(start 62.23 133.35)
-		(end 85.09 165.1)
+		(start 189.23 52.07)
+		(end 212.09 83.82)
 		(stroke
 			(width 0)
@@
 	(text "Mounting Hole Battery + LCD\n"
 		(exclude_from_sim no)
-		(at 74.422 130.556 0)
+		(at 201.422 49.276 0)
 		(effects
 			(font
@@
 	(text "M2 Screw"
 		(exclude_from_sim no)
-		(at 68.072 166.878 0)
+		(at 195.072 85.598 0)
 		(effects
 			(font
 				(size 1.27 1.27)
-			)
-		)
-	)
-	(text "Valider si j'ai pas inverser les connexion ici\ndu connecteur de la batterie\n"
-		(exclude_from_sim no)
-		(at 198.12 65.532 0)
-		(effects
-			(font
-				(size 1.524 1.524)
 			)
 		)
@@
 	(symbol
 		(lib_id "Mechanical:MountingHole")
-		(at 64.77 160.02 0)
+		(at 191.77 78.74 0)
 		(unit 1)
 		(exclude_from_sim yes)
@@
 		(fields_autoplaced yes)
 		(property "Reference" "H4"
-			(at 67.31 158.7499 0)
+			(at 194.31 77.4699 0)
 			(effects
 				(font
@@
 		)
 		(property "Value" "MountingHole"
-			(at 67.31 161.2899 0)
+			(at 194.31 80.0099 0)
 			(effects
 				(font
@@
 		)
 		(property "Footprint" "MountingHole:MountingHole_2.2mm_M2"
-			(at 64.77 160.02 0)
+			(at 191.77 78.74 0)
 			(effects
 				(font
@@
 		)
 		(property "Datasheet" "~"
-			(at 64.77 160.02 0)
+			(at 191.77 78.74 0)
 			(effects
 				(font
@@
 		)
 		(property "Description" "Mounting Hole without connection"
-			(at 64.77 160.02 0)
+			(at 191.77 78.74 0)
 			(effects
 				(font
@@
 	(symbol
 		(lib_id "Mechanical:MountingHole")
-		(at 64.77 152.4 0)
+		(at 191.77 71.12 0)
 		(unit 1)
 		(exclude_from_sim yes)
@@
 		(fields_autoplaced yes)
 		(property "Reference" "H3"
-			(at 67.31 151.1299 0)
+			(at 194.31 69.8499 0)
 			(effects
 				(font
@@
 		)
 		(property "Value" "MountingHole"
-			(at 67.31 153.6699 0)
+			(at 194.31 72.3899 0)
 			(effects
 				(font
@@
 		)
 		(property "Footprint" "MountingHole:MountingHole_2.2mm_M2"
-			(at 64.77 152.4 0)
+			(at 191.77 71.12 0)
 			(effects
 				(font
@@
 		)
 		(property "Datasheet" "~"
-			(at 64.77 152.4 0)
+			(at 191.77 71.12 0)
 			(effects
 				(font
@@
 		)
 		(property "Description" "Mounting Hole without connection"
-			(at 64.77 152.4 0)
+			(at 191.77 71.12 0)
 			(effects
 				(font
@@
 	(symbol
 		(lib_id "Mechanical:MountingHole")
-		(at 64.77 144.78 0)
+		(at 191.77 63.5 0)
 		(unit 1)
 		(exclude_from_sim yes)
@@
 		(fields_autoplaced yes)
 		(property "Reference" "H2"
-			(at 67.31 143.5099 0)
+			(at 194.31 62.2299 0)
 			(effects
 				(font
@@
 		)
 		(property "Value" "MountingHole"
-			(at 67.31 146.0499 0)
+			(at 194.31 64.7699 0)
 			(effects
 				(font
@@
 		)
 		(property "Footprint" "MountingHole:MountingHole_2.2mm_M2"
-			(at 64.77 144.78 0)
+			(at 191.77 63.5 0)
 			(effects
 				(font
@@
 		)
 		(property "Datasheet" "~"
-			(at 64.77 144.78 0)
+			(at 191.77 63.5 0)
 			(effects
 				(font
@@
 		)
 		(property "Description" "Mounting Hole without connection"
-			(at 64.77 144.78 0)
+			(at 191.77 63.5 0)
 			(effects
 				(font
@@
 	(symbol
 		(lib_id "Mechanical:MountingHole")
-		(at 64.77 137.16 0)
+		(at 191.77 55.88 0)
 		(unit 1)
 		(exclude_from_sim yes)
@@
 		(fields_autoplaced yes)
 		(property "Reference" "H1"
-			(at 67.31 135.8899 0)
+			(at 194.31 54.6099 0)
 			(effects
 				(font
@@
 		)
 		(property "Value" "MountingHole"
-			(at 67.31 138.4299 0)
+			(at 194.31 57.1499 0)
 			(effects
 				(font
@@
 		)
 		(property "Footprint" "MountingHole:MountingHole_2.2mm_M2"
-			(at 64.77 137.16 0)
+			(at 191.77 55.88 0)
 			(effects
 				(font
@@
 		)
 		(property "Datasheet" "~"
-			(at 64.77 137.16 0)
+			(at 191.77 55.88 0)
 			(effects
 				(font
@@
 		)
 		(property "Description" "Mounting Hole without connection"
-			(at 64.77 137.16 0)
-			(effects
-				(font
+			(at 191.77 55.88 0)
+			(effects
+				(font
