File: elec/Kicad/multimeter.kicad_sch (KiCad schematic)
At the start: 6 parts, among them J3 HX0201800000G

Commit message: multimetre final
Parts:
- added C5: 100nF, Capacitor_SMD:C_0603_1608Metric_Pad1.08x0.95mm_HandSolder, symbol Device:C
- added F2: F0603G0R03FNTR, F0603G0R03FNTR:F0603G0R03FNTR, symbol F0603G0R03FNTR:F0603G0R03FNTR
Connections:
- net GND: now also F2.2; no longer D4.C, D6.K
- net at J3.1: now also J3.2, R24.2
- net at J3.3: now also D4.A, D6.K, J3.4
- new net: C5.1, F2.1
- new net: C5.2, D4.C
Other:
- moved on the sheet: D6

Commit message: touillerie
Changed lines of the file:
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@@
 	)
 	(global_label "read_pin"
-		(shape input)
-		(at 36.83 29.21 0)
+		(shape output)
+		(at 36.83 29.21 90)
 		(fields_autoplaced yes)
 		(effects
@@
 		)
 		(property "Intersheetrefs" "${INTERSHEET_REFS}"
-			(at 47.8584 29.21 0)
+			(at 36.83 18.1816 90)
 			(effects
 				(font

Commit message: Jpense pas boire jeudi sérieux vue que y'a pas de 5@8
routage du découplage et des CLK
Parts:
- C5: footprint Capacitor_SMD:C_0603_1608Metric_Pad1.08x0.95mm_HandSolder -> Capacitor_SMD:C_0402_1005Metric_Pad0.74x0.62mm_HandSolder
- R22, R24: footprint Resistor_SMD:R_0603_1608Metric_Pad0.98x0.95mm_HandSolder -> Resistor_SMD:R_0402_1005Metric_Pad0.72x0.64mm_HandSolder
Changed lines of the file:
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@@
 	(paper "A4")
-	(junction
-		(at 26.67 111.76)
-		(diameter 0)
-		(color 0 0 0 0)
-	)
 	(junction
 		(at 41.91 125.73)
@@
 		(pts
 			(xy 69.85 82.55) (xy 69.85 95.25)
-		)
-		(stroke
-			(width 0)
-			(type default)
-		)
-	)
-	(wire
-		(pts
-			(xy 26.67 111.76) (xy 30.48 111.76)
 		)
 		(stroke
@@
 			)
 		)
-		(property "Footprint" "Capacitor_SMD:C_0603_1608Metric_Pad1.08x0.95mm_HandSolder"
+		(property "Footprint" "Capacitor_SMD:C_0402_1005Metric_Pad0.74x0.62mm_HandSolder"
 			(at 68.8848 82.55 0)
 			(effects
@@
 			)
 		)
-		(property "Footprint" "Resistor_SMD:R_0603_1608Metric_Pad0.98x0.95mm_HandSolder"
+		(property "Footprint" "Resistor_SMD:R_0402_1005Metric_Pad0.72x0.64mm_HandSolder"
 			(at 30.48 113.538 90)
 			(effects
@@
 			)
 		)
-		(property "Footprint" "Resistor_SMD:R_0603_1608Metric_Pad0.98x0.95mm_HandSolder"
+		(property "Footprint" "Resistor_SMD:R_0402_1005Metric_Pad0.72x0.64mm_HandSolder"
 			(at 35.052 118.11 90)
 			(effects

Commit message: jpense qu'on est ready to order
Other:
- moved on the sheet: C5, D4, D6, F1, F2, J3, R22, R24

Commit message: généré la schematic
Other:
- note added: "In Julien We Truss Que Ça Fonctionne"
- company: (none) -> University of Sherbrooke
- title: (none) -> Touillomètre - Multimeter
Changed lines of the file:
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@@
 	(generator_version "8.0")
 	(paper "A4")
+	(title_block
+		(title "Touillomètre - Multimeter")
+		(date "2024-12-26")
+		(rev "C3I")
+		(company "University of Sherbrooke")
+	)
 	(junction
 		(at 71.12 30.48)
@@
 		)
 	)
+	(text "In Julien We Truss Que Ça Fonctionne"
+		(exclude_from_sim no)
+		(at 62.484 20.32 0)
+		(effects
+			(font
+				(size 2.54 2.54)
+				(thickness 0.508)
+				(bold yes)
+			)
+		)
+	)
